Commit message: First movement of wheels

File: src/URDF/cyberpod.urdf (robot description, URDF)
Before this commit: robot cyberpod, 3 links, 2 joints
Links:
- link cyberpod/base_link: mass 1 -> 0.001
Joints:
- joint w1_joint: axis (none) -> 0 1 0; type fixed -> continuous
- joint w2_joint: axis (none) -> 0 1 0; type fixed -> continuous

Commit message: Modify inertia to get more realistic

File: src/URDF/cyberpod.urdf (robot description, URDF)
Before this commit: robot cyberpod, 3 links, 2 joints
Links:
- link cyberpod/base_link: mass 0.001 -> 1
